File: LS4_FLYBACK.kicad_sch (KiCad schematic)
At the start: 14 parts, among them U4 VNLD5160TR-E, U5 VNLD5160TR-E

Commit message: Export rev-e
Parts:
- added D1, D10, D15, D2, D42, D5: B5819W, hellen-one-common:SOD-123, symbol hellen-one-common:1N4148WS
- added R13, R2, R43, R44, R45, R5, R50, R61, R83, R84, R95, R97: 4.7k, hellen-one-common:R0603, symbol hellen-one-common:Res
- added U12, U3, U7: VNLD5160TR-E, Package_SO:SOIC-8_3.9x4.9mm_P1.27mm, symbol chips:VNLD5160
- gave numbers to parts that had none: 4
- renumbered R30 to R73, R30 to R74, R30 to R75, R30 to R77
Connections:
- net 12V_FLYBACK: now also D1.1 (K), D10.1 (K), D15.1 (K), D2.1 (K), D42.1 (K), D5.1 (K)
- net GND: now also R44.1, R45.1, R50.1, R61.1, R95.1, R97.1, U12.5 (S2), U12.7 (S1), U3.5 (S2), U3.7 (S1), U7.5 (S2), U7.7 (S1)
- new net: R83.1, U12.1 (IN1)
- new net: R13.1, U7.1 (IN1)
- new net: R5.1, U3.3 (IN2)
- new net: R2.1, U3.1 (IN1)
- new net: R43.1, U7.3 (IN2)
- new net: R84.1, U12.3 (IN2)
- new net IN10: R84.2, R95.2
- new net IN5: R2.2, R50.2
- new net IN6: R44.2, R5.2
- new net IN7: R13.2, R61.2
- new net IN8: R43.2, R45.2
- new net IN9: R83.2, R97.2
- new net OUT10: D42.2 (A), U12.6 (D2)
- new net OUT5: D1.2 (A), U3.8 (D1)
- new net OUT6: D2.2 (A), U3.6 (D2)
- new net OUT7: D5.2 (A), U7.8 (D1)
- new net OUT8: D10.2 (A), U7.6 (D2)
- new net OUT9: D15.2 (A), U12.8 (D1)
- no-connect marks 4 -> 10
Other:
- company: rusefi.com -> rusEFI
- title: (none) -> hellen154hyundai
- moved on the sheet: D27, R41, R42, R48, R49, R73, R74, R75, R77, U4, U5
