File: LS6.kicad_sch (KiCad schematic)
At the start: 15 parts, among them U1 VNLD5160TR-E, U2 VNLD5160TR-E, U6 VNLD5160TR-E

Commit message: Export rev-e
Parts:
- gave numbers to parts that had none: 12
Other:
- company: rusefi.com -> rusEFI
- title: (none) -> hellen154hyundai
